File: Lithium_Board.kicad_sch (KiCad schematic)
At the start: 67 parts, among them IC1 BQ25750RRVR, IC2 TPS70933DBVR, J1 XT30PW-M, J2 XT30PW-F, J3 XT30PW-M, J5 TSW-105-07-G-S, Q1 SIR870ADP-T1-GE3, Q2 SIR870ADP-T1-GE3, Q3 SIR870ADP-T1-GE3, Q4 SIR870ADP-T1-GE3, Q5 SIR870ADP-T1-GE3, Q6 SIR870ADP-T1-GE3, Q7 SIR870ADP-T1-GE3, Q8 SIR870ADP-T1-GE3

Commit message: Small Changes
Parts:
- added C29: 100nF [HV], C0603C104K1RACAUTO:CAPC1608X95N, symbol C0603C104K1RACAUTO:C0603C104K1RACAUTO
- added C30: 4.7uF [HV], KAM32LR72A475KU:CAPC3225X94N, symbol KAM32LR72A475KU:KAM32LR72A475KU
Connections:
- net GND: now also C29.2, C30.2
- net +48V renamed VIN
- net VIN: now also C29.1, C30.1
Other:
- note added: "INPUT CAPACITORS"
- moved on the sheet: C1

Commit message: First Big Review Changes
Parts:
- removed IC2: TPS70933DBVR, TPS70933DBVR:SOT95P280X145-5N, symbol TPS70933DBVR:TPS70933DBVR
- removed R11: 249k, RC0603FR-07249KL:RESC1608X55N, symbol RC0603FR-07249KL:RC0603FR-07249KL
- removed R25: 34.8k, RC0603FR-0734K8L:RESC1608X55N, symbol RC0603FR-0734K8L:RC0603FR-0734K8L
- added IC2: TPS70933DRVR, SON65P200X200X80-7N, symbol TPS70933DRVR:TPS70933DRVR
- added R11: 249kΩ, RESC1608X55N, symbol RT0603BRD07249KL:RT0603BRD07249KL
- added R25: 35.2kΩ, RESC1608X55N, symbol RT0603BRD0735K2L:RT0603BRD0735K2L
- D2, D5: footprint SODFL3516X100N -> CDBMT2100-HF:SODFL3516X100N
Connections:
- net +3V3: now also IC2.1 (OUT)
- net +BATT: now also IC2.6 (IN), R11.2
- net BQ_FB: now also R11.1, R25.1
- net FBG: now also R25.2
- net GND: now also IC2.3 (GND_1), IC2.7 (GND_2)
- no-connect marks 8 -> 10
Other:
- moved on the sheet: C16, C17

Commit message: Fixed Big Capacitor
Parts:
- removed C23: EEV-FK2A101V, EEV-FK2A101V:EEEFK0J682AV, symbol EEV-FK2A101V:EEV-FK2A101V
- added C23: EEE-TP1K391V, EEE-TP1K391V:EEEFK0J682AV, symbol EEE-TP1K391V:EEE-TP1K391V
- IC2: footprint SON65P200X200X80-7N -> TPS70933DRVR:SON65P200X200X80-7N
Connections:
- net BQ_SYS: now also C23.1 (+_1), C23.3 (+_2), C23.4 (+_3)
- net GND: now also C23.2 (-_1), C23.5 (-_2), C23.6 (-_3)
Changed lines of the file:
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@@
-	)
-	(symbol
-		(lib_id "EEV-FK2A101V:EEV-FK2A101V")
-		(at 190.5 265.43 180)
-		(unit 1)
-		(exclude_from_sim no)
-		(in_bom yes)
-		(on_board yes)
-		(dnp no)
-		(property "Reference" "C23"
-			(at 197.358 257.556 0)
-			(effects
-				(font
-					(size 1.27 1.27)
-				)
-				(justify right)
-			)
-		)
-		(property "Value" "EEV-FK2A101V"
-			(at 192.278 260.096 0)
-			(effects
-				(font
-					(size 1.27 1.27)
-				)
-				(justify right)
-			)
-		)
-		(property "Footprint" "EEV-FK2A101V:EEEFK0J682AV"
-			(at 168.91 178.13 0)
-			(effects
-				(font
-					(size 1.27 1.27)
-				)
-				(justify left top)
-				(hide yes)
-			)
-		)
-		(property "Datasheet" "http://industrial.panasonic.com/cdbs/www-data/pdf/RDE0000/ABA0000C1181.pdf"
-			(at 168.91 78.13 0)
-			(effects
-				(font
-					(size 1.27 1.27)
-				)
-				(justify left top)
-				(hide yes)
-			)
-		)
-		(property "Description" "Aluminium Electroyltic Capacitor, Radial, Vibration-Proof"
-			(at 190.5 265.43 0)
-			(effects
-				(font
-					(size 1.27 1.27)
-				)
-				(hide yes)
-			)
-		)
-		(property "Height" "16.8"
-			(at 168.91 -121.87 0)
-			(effects
-				(font
-					(size 1.27 1.27)
-				)
-				(justify left top)
-				(hide yes)
-			)
-		)
-		(property "Mouser Part Number" "667-EEV-FK2A101V"
-			(at 168.91 -221.87 0)
-			(effects
-				(font
-					(size 1.27 1.27)
-				)
-				(justify left top)
-				(hide yes)
-			)
-		)
-		(property "Mouser Price/Stock" "https://www.mouser.co.uk/ProductDetail/Panasonic/EEV-FK2A101V?qs=MtOUKumLmnaVkoWQWMGNWA%3D%3D"
-			(at 168.91 -321.87 0)
-			(effects
-				(font
-					(size 1.27 1.27)
-				)
-				(justify left top)
-				(hide yes)
-			)
-		)
-		(property "Manufacturer_Name" "Panasonic"
-			(at 168.91 -421.87 0)
-			(effects
-				(font
-					(size 1.27 1.27)
-				)
-				(justify left top)
-				(hide yes)
-			)
-		)
-		(property "Manufacturer_Part_Number" "EEV-FK2A101V"
-			(at 168.91 -521.87 0)
-			(effects
-				(font
-					(size 1.27 1.27)
-				)
-				(justify left top)
-				(hide yes)
-			)
-		)
-		(pin "2"
-		)
-		(pin "4"
-		)
-		(pin "1"
-		)
-		(pin "3"
-		)
-		(pin "6"
-		)
-		(pin "5"
-		)
-		(instances
-			(project ""
-				(path "/a208389b-7ee7-48d8-95f2-b3e129849547"
-					(reference "C23")
-					(unit 1)
-				)
-			)
-		)
 	)
 	(symbol
@@
 			)
 		)
-		(property "Footprint" "SON65P200X200X80-7N"
+		(property "Footprint" "TPS70933DRVR:SON65P200X200X80-7N"
 			(at 383.54 352.73 0)
 			(effects
@@
 					(unit 1)
 				)
+			)
+		)
+	)
+	(symbol
+		(lib_id "EEE-TP1K391V:EEE-TP1K391V")
+		(at 190.5 265.43 180)
+		(unit 1)
+		(exclude_from_sim no)
+		(in_bom yes)
+		(on_board yes)
+		(dnp no)
+		(property "Reference" "C23"
+			(at 198.12 256.794 0)
+			(effects
+				(font
+					(size 1.27 1.27)
+				)
+				(justify right)
+			)
+		)
+		(property "Value" "EEE-TP1K391V"
+			(at 193.802 259.588 0)
+			(effects
+				(font
+					(size 1.27 1.27)
+				)
+				(justify right)
+			)
+		)
+		(property "Footprint" "EEE-TP1K391V:EEEFK0J682AV"
+			(at 168.91 178.13 0)
+			(effects
+				(font
+					(size 1.27 1.27)
+				)
+				(justify left top)
+				(hide yes)
+			)
+		)
+		(property "Datasheet" "http://industrial.panasonic.com/cdbs/www-data/pdf/RDE0000/RDE0000C1255.pdf"
+			(at 168.91 78.13 0)
+			(effects
+				(font
+					(size 1.27 1.27)
+				)
+				(justify left top)
+				(hide yes)
+			)
+		)
+		(property "Description" "Aluminum Electrolytic Capacitors - SMD 80VDC 390uF 20% SMD AEC-Q200 Vibe Proof"
+			(at 190.5 265.43 0)
+			(effects
+				(font
+					(size 1.27 1.27)
+				)
+				(hide yes)
+			)
+		)
+		(property "Height" "16.8"
+			(at 168.91 -121.87 0)
+			(effects
+				(font
+					(size 1.27 1.27)
+				)
+				(justify left top)
+				(hide yes)
+			)
+		)
+		(property "Mouser Part Number" "667-EEE-TP1K391V"
+			(at 168.91 -221.87 0)
+			(effects
+				(font
+					(size 1.27 1.27)
+				)
+				(justify left top)
+				(hide yes)
+			)
+		)
+		(property "Mouser Price/Stock" "https://www.mouser.co.uk/ProductDetail/Panasonic/EEE-TP1K391V?qs=XFmntM7Yc9dUeO1BN5vyvw%3D%3D"
+			(at 168.91 -321.87 0)
+			(effects
+				(font
+					(size 1.27 1.27)
+				)
+				(justify left top)
+				(hide yes)
+			)
+		)
+		(property "Manufacturer_Name" "Panasonic"
+			(at 168.91 -421.87 0)
+			(effects
+				(font
+					(size 1.27 1.27)
+				)
+				(justify left top)
+				(hide yes)
+			)
+		)
+		(property "Manufacturer_Part_Number" "EEE-TP1K391V"
+			(at 168.91 -521.87 0)
+			(effects
+				(font
+					(size 1.27 1.27)
+				)
+				(justify left top)
+				(hide yes)
+			)
+		)
+		(pin "5"
+		)
+		(pin "3"
+		)
+		(pin "6"
+		)
+		(pin "4"
+		)
+		(pin "2"
+		)
+		(pin "1"
+		)
+		(instances
+			(project ""
+				(path "/a208389b-7ee7-48d8-95f2-b3e129849547"
+					(reference "C23")
+					(unit 1)
+				)

Commit message: Final Changes+Stackup Fixed
Parts:
- removed C16: 1uF, C2012X7R1H105K125AB:CAPC2012X145N, symbol C2012X7R1H105K125AB:C2012X7R1H105K125AB
- removed C8: 100uF, EEE-FT1V101AP:EEE1AA101SP, symbol EEE-FT1V101AP:EEE-FT1V101AP
- removed IC2: TPS70933DRVR, TPS70933DRVR:SON65P200X200X80-7N, symbol TPS70933DRVR:TPS70933DRVR
- added C16: 4.7uF, UMJ325AB7475KMHP:CAPC3225X280N, symbol UMJ325AB7475KMHP:UMJ325AB7475KMHP
- added C8: 150uF, EEEHP1H4R7P, symbol EEH-ZL1E151P:EEH-ZL1E151P
- added IC2: MCP1792T-3302H_DB, MCP1792T-3302H_DB:SOT230P700X180-4N, symbol MCP1792T-3302H_DB:MCP1792T-3302H_DB
- C23: value EEE-TP1K391V -> 390uF
- R11: footprint RESC1608X55N -> RT0603BRD07249KL:RESC1608X55N
- R25: footprint RESC1608X55N -> RT0603BRD0735K2L:RESC1608X55N
Connections:
- net +3V3: now also IC2.3 (VOUT)
- net +BATT: now also C16.1, IC2.1 (VIN)
- net GND: now also C16.2, C8.2 (-), IC2.2 (GND_1), IC2.4 (GND_2)
- net Q7_DRAIN: now also C8.1 (+)
- no-connect marks 10 -> 7
Other:
- note added: "25V"
- note added: "80V"
- note removed: "35V"

Commit message: Fixed Items Not in Stock
Parts:
- C8: footprint EEEHP1H4R7P -> EEH-ZL1E151P:EEEHP1H4R7P
Changed lines of the file:
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@@
 			)
 		)
-		(property "Footprint" "EEEHP1H4R7P"
+		(property "Footprint" "EEH-ZL1E151P:EEEHP1H4R7P"
 			(at 390.22 138.43 0)
 			(effects
