File: CANBUS.kicad_sch (KiCad schematic)
At the start: 10 parts, among them IC5 TCAN3414DR, J4 S3B-XH-SM4-TB_LF__SN_

Commit message: Fixed Items Not in Stock
Parts:
- removed D1: CDSOT23-T24CAN, CDSOT23-T24CAN:SOT95P230X117-3N, symbol CDSOT23-T24CAN:CDSOT23-T24CAN
- removed IC5: TCAN3414DR, TCAN3414DR:SOIC127P600X175-8N, symbol TCAN3414DR:TCAN3414DR
- added D1: ESDCAN24-2BLY, SOT95P255X125-3N, symbol ESDCAN24-2BLY:ESDCAN24-2BLY
- added IC3: TCAN3414DDFR, INA190A2NDDFREP, symbol TCAN3414DDFR:TCAN3414DDFR
Connections:
- net +3V3: now also IC3.3 (VCC)
- net CAN_N: now also D1.1 (I/O_1)
- net CAN_P: now also D1.2 (I/O_2)
- net CAN_STB: now also IC3.8 (STB)
- net FDCAN_RX: now also IC3.4 (RXD)
- net FDCAN_TX: now also IC3.1 (TXD)
- net GND: now also D1.3 (I/O_3), IC3.2 (GND), IC3.5 (SHDNVIO)
- net L_CAN_N: now also IC3.6 (CANL)
- net L_CAN_P: now also IC3.7 (CANH)

Commit message: New BOM+GRB
Parts:
- D1: footprint SOT95P255X125-3N -> ESDCAN24-2BLY:SOT95P255X125-3N
- IC3: footprint INA190A2NDDFREP -> TCAN3414DDFR:INA190A2NDDFREP
Changed lines of the file:
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@@
 			)
 		)
-		(property "Footprint" "INA190A2NDDFREP"
+		(property "Footprint" "TCAN3414DDFR:INA190A2NDDFREP"
 			(at 107.95 162.23 0)
 			(effects
@@
 			)
 		)
-		(property "Footprint" "SOT95P255X125-3N"
+		(property "Footprint" "ESDCAN24-2BLY:SOT95P255X125-3N"
 			(at 196.85 -22.53 0)
 			(effects
