File: mcu.kicad_sch (KiCad schematic)
At the start: 9 parts, among them IC4 STM32G0B1CBT6N

Commit message: Final Changes+Stackup Fixed
Parts:
- added C31: 4.7uF, UMJ325AB7475KMHP:CAPC3225X280N, symbol UMJ325AB7475KMHP:UMJ325AB7475KMHP
Connections:
- net +3V3: now also C31.1
- net GND: now also C31.2

Commit message: Fixed Items Not in Stock
Parts:
- removed IC4: STM32G0B1CBT6N, STM32G0B1CBT6N:QFP50P900X900X160-48N, symbol STM32G0B1CBT6N:STM32G0B1CBT6N
- added IC4: STM32G0B1CET6N, QFP50P900X900X160-48N, symbol STM32G0B1CET6N:STM32G0B1CET6N
Connections:
- net +3V3: now also IC4.31 (VDDIO2), IC4.4 (VBAT), IC4.5 (VREF+), IC4.6 (VDD/VDDA)
- net BQ2_ALERT: now also IC4.15 (PA4)
- net BQ2_CS: now also IC4.24 (PB12)
- net BQ2_MISO: now also IC4.17 (PA6)
- net BQ2_MOSI: now also IC4.18 (PA7)
- net BQ2_SCLK: now also IC4.16 (PA5)
- net BQ_CE: now also IC4.13 (PA2)
- net BQ_INT: now also IC4.11 (PA0)
- net BQ_PG: now also IC4.12 (PA1)
- net BQ_SCL: now also IC4.45 (PB6)
- net BQ_SDA: now also IC4.46 (PB7)
- net BQ_STAT1: now also IC4.19 (PB0)
- net BQ_STAT2: now also IC4.20 (PB1)
- net CAN_STB: now also IC4.14 (PA3)
- net FDCAN_RX: now also IC4.47 (PB8)
- net FDCAN_TX: now also IC4.48 (PB9)
- net GND: now also IC4.30 (VSS), IC4.7 (VSS/VSSA)
- net LED1_RED: now also IC4.28 (PA8)
- net LED2_GREEN: now also IC4.29 (PA9)
- net NRST: now also IC4.10 (PF2-NRST)
- net SWCLK: now also IC4.36 (PA14-BOOT0)
- net SWDIO: now also IC4.35 (PA13)
Changed lines of the file:
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@@
+	)
+	(symbol
+		(lib_id "STM32G0B1CET6N:STM32G0B1CET6N")
+		(at 116.84 54.61 0)
+		(unit 1)
+		(exclude_from_sim no)
+		(in_bom yes)
+		(on_board yes)
+		(dnp no)
+		(fields_autoplaced yes)
+		(property "Reference" "IC4"
+			(at 172.72 48.1898 0)
+			(effects
+				(font
+					(size 1.27 1.27)
+				)
+			)
+		)
+		(property "Value" "STM32G0B1CET6N"
+			(at 172.72 50.7298 0)
+			(effects
+				(font
+					(size 1.27 1.27)
+				)
+			)
+		)
+		(property "Footprint" "QFP50P900X900X160-48N"
+			(at 163.83 141.91 0)
+			(effects
+				(font
+					(size 1.27 1.27)
+				)
+				(justify left top)
+				(hide yes)
+			)
+		)
+		(property "Datasheet" "https://www.st.com/resource/en/datasheet/stm32g0b1cc.pdf"
+			(at 163.83 241.91 0)
+			(effects
+				(font
+					(size 1.27 1.27)
+				)
+				(justify left top)
+				(hide yes)
+			)
+		)
+		(property "Description" "Mainstream Arm Cortex-M0+ 32-bit MCU, up to 512KB Flash, 144KB RAM, 6x USART, timers, ADC, DAC, comm. I/Fs, 1.7-3.6V"
+			(at 116.84 54.61 0)
+			(effects
+				(font
+					(size 1.27 1.27)
+				)
+				(hide yes)
+			)
+		)
+		(property "Height" "1.6"
+			(at 163.83 441.91 0)
+			(effects
+				(font
+					(size 1.27 1.27)
+				)
+				(justify left top)
+				(hide yes)
+			)
+		)
+		(property "Mouser Part Number" "511-STM32G0B1CET6N"
+			(at 163.83 541.91 0)
+			(effects
+				(font
+					(size 1.27 1.27)
+				)
+				(justify left top)
+				(hide yes)
+			)
+		)
+		(property "Mouser Price/Stock" "https://www.mouser.co.uk/ProductDetail/STMicroelectronics/STM32G0B1CET6N?qs=CiayqK2gdcK2xI5l7E1NcQ%3D%3D"
+			(at 163.83 641.91 0)
+			(effects
+				(font
+					(size 1.27 1.27)
+				)
+				(justify left top)
+				(hide yes)
+			)
+		)
+		(property "Manufacturer_Name" "STMicroelectronics"
+			(at 163.83 741.91 0)
+			(effects
+				(font
+					(size 1.27 1.27)
+				)
+				(justify left top)
+				(hide yes)
+			)
+		)
+		(property "Manufacturer_Part_Number" "STM32G0B1CET6N"
+			(at 163.83 841.91 0)
+			(effects
+				(font
+					(size 1.27 1.27)
+				)
+				(justify left top)
+				(hide yes)
+			)
+		)
+		(pin "34"
+		)
+		(pin "32"
+		)
+		(pin "33"
+		)
+		(pin "17"
+		)
+		(pin "44"
+		)
+		(pin "16"
+		)
+		(pin "45"
+		)
+		(pin "15"
+		)
+		(pin "46"
+		)
+		(pin "47"
+		)
+		(pin "13"
+		)
+		(pin "48"
+		)
+		(pin "12"
+		)
+		(pin "11"
+		)
+		(pin "10"
+		)
+		(pin "9"
+		)
+		(pin "8"
+		)
+		(pin "7"
+		)
+		(pin "6"
+		)
+		(pin "5"
+		)
+		(pin "4"
+		)
+		(pin "3"
+		)
+		(pin "2"
+		)
+		(pin "1"
+		)
+		(pin "14"
+		)
+		(pin "31"
+		)
+		(pin "30"
+		)
+		(pin "29"
+		)
+		(pin "28"
+		)
+		(pin "27"
+		)
+		(pin "26"
+		)
+		(pin "25"
+		)
+		(pin "35"
+		)
+		(pin "36"
+		)
+		(pin "37"
+		)
+		(pin "24"
+		)
+		(pin "23"
+		)
+		(pin "21"
+		)
+		(pin "39"
+		)
+		(pin "22"
+		)
+		(pin "38"
+		)
+		(pin "40"
+		)
+		(pin "42"
+		)
+		(pin "19"
+		)
+		(pin "41"
+		)
+		(pin "20"
+		)
+		(pin "18"
+		)
+		(pin "43"
+		)
+		(instances
+			(project ""
+				(path "/a208389b-7ee7-48d8-95f2-b3e129849547/160492a7-828d-4540-9766-a6c613c08096"
+					(reference "IC4")
+					(unit 1)
+				)
+			)
+		)
 	)
 	(symbol
@@
 					(unit 1)
 				)
-			)
-		)
-	)
-	(symbol
-		(lib_id "STM32G0B1CBT6N:STM32G0B1CBT6N")
-		(at 116.84 54.61 0)
-		(unit 1)
-		(exclude_from_sim no)
-		(in_bom yes)
-		(on_board yes)
-		(dnp no)
-		(fields_autoplaced yes)
-		(property "Reference" "IC4"
-			(at 172.72 48.1898 0)
-			(effects
-				(font
-					(size 1.27 1.27)
-				)
-			)
-		)
-		(property "Value" "STM32G0B1CBT6N"
-			(at 172.72 50.7298 0)
-			(effects
-				(font
-					(size 1.27 1.27)
-				)
-			)
-		)
-		(property "Footprint" "STM32G0B1CBT6N:QFP50P900X900X160-48N"
-			(at 163.83 141.91 0)
-			(effects
-				(font
-					(size 1.27 1.27)
-				)
-				(justify left top)
-				(hide yes)
-			)
-		)
-		(property "Datasheet" "https://www.st.com/resource/en/datasheet/stm32g0b1cc.pdf"
-			(at 163.83 241.91 0)
-			(effects
-				(font
-					(size 1.27 1.27)
-				)
-				(justify left top)
-				(hide yes)
-			)
-		)
-		(property "Description" "Mainstream Arm Cortex-M0+ 32-bit MCU, up to 128KB Flash, 144KB RAM, 6x USART, timers, ADC, DAC, comm. I/Fs, 1.7-3.6V"
-			(at 116.84 54.61 0)
-			(effects
-				(font
-					(size 1.27 1.27)
-				)
-				(hide yes)
-			)
-		)
-		(property "Height" "1.6"
-			(at 163.83 441.91 0)
-			(effects
-				(font
-					(size 1.27 1.27)
-				)
-				(justify left top)
-				(hide yes)
-			)
-		)
-		(property "Mouser Part Number" "511-STM32G0B1CBT6N"
-			(at 163.83 541.91 0)
-			(effects
-				(font
-					(size 1.27 1.27)
-				)
-				(justify left top)
-				(hide yes)
-			)
-		)
-		(property "Mouser Price/Stock" "https://www.mouser.co.uk/ProductDetail/STMicroelectronics/STM32G0B1CBT6N?qs=CiayqK2gdcI7R4IDpukH4w%3D%3D"
-			(at 163.83 641.91 0)
-			(effects
-				(font
-					(size 1.27 1.27)
-				)
-				(justify left top)
-				(hide yes)
-			)
-		)
-		(property "Manufacturer_Name" "STMicroelectronics"
-			(at 163.83 741.91 0)
-			(effects
-				(font
-					(size 1.27 1.27)
-				)
-				(justify left top)
-				(hide yes)
-			)
-		)
-		(property "Manufacturer_Part_Number" "STM32G0B1CBT6N"
-			(at 163.83 841.91 0)
-			(effects
-				(font
-					(size 1.27 1.27)
-				)
-				(justify left top)
-				(hide yes)
-			)
-		)
-		(pin "39"
-		)
-		(pin "22"
-		)
-		(pin "21"
-		)
-		(pin "38"
-		)
-		(pin "23"
-		)
-		(pin "37"
-		)
-		(pin "24"
-		)
-		(pin "36"
-		)
-		(pin "35"
-		)
-		(pin "34"
-		)
-		(pin "33"
-		)
-		(pin "32"
-		)
-		(pin "31"
-		)
-		(pin "30"
-		)
-		(pin "29"
-		)
-		(pin "28"
-		)
-		(pin "27"
-		)
-		(pin "26"
-		)
-		(pin "25"
-		)
-		(pin "40"
-		)
-		(pin "20"
-		)
-		(pin "5"
-		)
-		(pin "3"
-		)
-		(pin "4"
-		)
-		(pin "2"
-		)
-		(pin "1"
-		)
-		(pin "7"
-		)
-		(pin "6"
-		)
-		(pin "15"
-		)
-		(pin "8"
-		)
-		(pin "9"
-		)
-		(pin "45"
-		)
-		(pin "11"
-		)
-		(pin "41"
-		)
-		(pin "12"
-		)
-		(pin "48"
-		)
-		(pin "47"
-		)
-		(pin "13"
-		)
-		(pin "14"
-		)
-		(pin "42"
-		)
-		(pin "46"
-		)
-		(pin "10"
-		)
-		(pin "18"
-		)
-		(pin "43"
-		)
-		(pin "17"
-		)
-		(pin "44"
-		)
-		(pin "16"
-		)
-		(pin "19"
-		)
-		(instances
-			(project ""
-				(path "/a208389b-7ee7-48d8-95f2-b3e129849547/160492a7-828d-4540-9766-a6c613c08096"
-					(reference "IC4")
-					(unit 1)
-				)

Commit message: New BOM+GRB
Parts:
- IC4: footprint QFP50P900X900X160-48N -> STM32G0B1CET6N:QFP50P900X900X160-48N
Changed lines of the file:
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@@
 			)
 		)
-		(property "Footprint" "QFP50P900X900X160-48N"
+		(property "Footprint" "STM32G0B1CET6N:QFP50P900X900X160-48N"
 			(at 163.83 141.91 0)
 			(effects

Commit message: BOM Fixed+CS Fixed
Connections:
- net BQ2_CS: now also IC4.37 (PA15); no longer IC4.24 (PB12)
Changed lines of the file:
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@@
+	)
+	(no_connect
+		(at 154.94 97.79)
 	)
 	(no_connect
@@
 	)
 	(no_connect
-		(at 154.94 39.37)
-	)
-	(no_connect
 		(at 116.84 59.69)
 	)
@@
 		)
 	)
+	(global_label "LED1_RED"
+		(shape input)
+		(at 81.28 149.86 0)
+		(fields_autoplaced yes)
+		(effects
+			(font
+				(size 1.27 1.27)
+			)
+			(justify left)
+		)
+		(property "Intersheetrefs" "${INTERSHEET_REFS}"
+			(at 93.5784 149.86 0)
+			(effects
+				(font
+					(size 1.27 1.27)
+				)
+				(justify left)
+				(hide yes)
+			)
+		)
+	)
 	(global_label "BQ2_CS"
 		(shape input)
-		(at 154.94 97.79 270)
-		(fields_autoplaced yes)
-		(effects
-			(font
-				(size 1.27 1.27)
-			)
-			(justify right)
-		)
-		(property "Intersheetrefs" "${INTERSHEET_REFS}"
-			(at 154.94 108.0323 90)
-			(effects
-				(font
-					(size 1.27 1.27)
-				)
-				(justify right)
-				(hide yes)
-			)
-		)
-	)
-	(global_label "LED1_RED"
-		(shape input)
-		(at 81.28 149.86 0)
+		(at 154.94 39.37 90)
 		(fields_autoplaced yes)
 		(effects
@@
 		)
 		(property "Intersheetrefs" "${INTERSHEET_REFS}"
-			(at 93.5784 149.86 0)
-			(effects
-				(font
+			(at 154.94 29.1277 90)
+			(effects
+				(font
